File: rtc_temp_switch.sch (KiCad schematic (older format))
At the start: 14 parts, among them SW1 SW_Push, SW2 SW_Push, U2 MCP7940N-xST, U7 LM35-LP, Y1 32,768kHz

Commit message: małe poprawki podczas montażu
Connections:
- net 12V is gone; now on net 5V: U7.3 (GND)
Changed lines of the file:
@@
 Wire Wire Line
 	3900 5050 4200 5050
-Text HLabel 4200 5350 0    50   Input ~ 0
-12V
 Wire Wire Line
 	4200 5350 4450 5350
 Wire Wire Line
 	4450 5350 4450 5450
+Text HLabel 4200 5350 0    50   Input ~ 0
+5V
 $EndSCHEMATC
