File: ni12_zegar.kicad_pcb (KiCad board)
At the start: 2 copper layers, 100 x 100 mm, 153 parts, among them IC1 MAX1771, J1 Jack-DC, Q1 IRF740, Q10 MPSA92, Q11 MPSA92, Q12 MPSA92, Q13 MPSA92, Q14 MPSA92, Q15 MPSA92, Q16 MPSA92, Q17 MPSA92, Q18 MPSA92, Q19 MPSA92, Q2 MPSA92, Q20 MPSA92, Q21 MPSA92, Q22 MPSA92, Q23 MPSA92, Q24 MPSA92, Q25 MPSA92, Q26 MPSA92, Q27 MPSA92, Q28 MPSA92, Q29 MPSA92, Q3 MPSA92, Q30 MPSA92, Q31 MPSA92, Q32 MPSA92, Q33 MPSA92, Q34 MPSA92, Q35 MPSA92, Q36 MPSA92, Q37 MPSA92, Q38 MPSA92, Q39 MPSA92, Q4 MPSA92, Q40 MPSA92, Q41 MPSA92, Q42 MPSA92, Q5 MPSA92, Q6 MPSA92, Q7 MPSA92, Q8 MPSA92, Q9 MPSA92, SW1 SW_Push, SW2 SW_Push, U1 L7805, U2 MCP7940N-xST, U3 4028, U4 4028, U5 4028, U6 4028, U7 LM35-LP, Y1 32,768kHz

Commit message: małe poprawki podczas montażu
Connections:
- A1 pad 17: Net-(A1-Pad17) -> (no net)
- A1 pad 18: Net-(A1-Pad18) -> (no net)
- A1 pad 27: Net-(A1-Pad27) -> (no net)
- A1 pad 28: Net-(A1-Pad28) -> (no net)
- A1 pad 3: Net-(A1-Pad3) -> (no net)
- U7 pad 3: /12V -> /5V
Routing:
- net /12V: track 102.9 -> 86.5 mm
- net /5V: track 161.6 -> 172.8 mm
- net /sw2: vias 1 -> 0

Commit message: drobne poprawki
Connections:
- A1 pad 22: /sw1 -> /neon
- A1 pad 23: /neon -> /SDA
- A1 pad 25: /SDA -> /sw1
Routing:
- net /SDA: track 31.5 -> 43.9 mm
- net /sw1: track 11.9 -> 18.9 mm
- net /neon: track 61.4 -> 63.9 mm
- net /rtc/MPF: track 14.7 -> 14.1 mm
- net GND: vias 310 -> 391
