File: ni12_zegar.sch (KiCad schematic (older format))
At the start: 7 parts

Commit message: drobne poprawki
Connections:
- net SDA: now also A1.23 (A4); no longer A1.25 (A6)
- net neon: now also A1.22 (A3); no longer A1.23 (A4)
- net sw1: now also A1.25 (A6); no longer A1.22 (A3)
Changed lines of the file:
@@
 	3950 1650 4500 1650
 Connection ~ 4500 1650
-Text Label 8350 2450 0    50   ~ 0
+Text Label 8400 2450 2    50   ~ 0
 SCL
-Text Label 8350 2550 0    50   ~ 0
+Text Label 8400 2350 2    50   ~ 0
 SDA
 Wire Wire Line
-	8350 2450 8150 2450
-Wire Wire Line
-	8150 2550 8350 2550
+	8400 2450 8150 2450
+Wire Wire Line
+	8150 2550 8400 2550
 $Comp
 L power:GND #PWR01
@@
 Text Label 6000 3950 2    50   ~ 0
 neon
-Text Label 8400 2350 2    50   ~ 0
+Text Label 8450 2250 2    50   ~ 0
 neon
 Wire Wire Line
@@
 	8150 2350 8400 2350
 Wire Wire Line
-	8150 2650 8350 2650
+	8150 2650 8400 2650
 Wire Wire Line
 	8150 2150 8450 2150
@@
 Text Label 8450 2150 2    50   ~ 0
 sw2
-Text Label 8450 2250 2    50   ~ 0
+Text Label 8400 2550 2    50   ~ 0
 sw1
-Text Label 8350 2650 2    50   ~ 0
+Text Label 8400 2650 2    50   ~ 0
 temp
 Wire Wire Line
